File: uOsc_1_v3.sch (EAGLE design)
At the start: 101 parts, among them IC10 TL072, IC3 LM4040B25, IC4 MCP3204-TSSOP-14, IC5 DAC8551, IC6 LM1117-3.3, IC7 MCP6004, IC8 LM4040B10, IC9 TL074, J1 S_JACK_S2_INV, J2 S_JACK_S2_INV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

Commit message: uOsc-I files
Other:
- note added: "Codex-Modulex"
- note added: "Original design by: Olivier Gillet of Mutable Instruments"
- note added: "info@codex-modulex.com"
- note removed: "Olivier Gillet"
- note removed: "ol.gillet@gmail.com"
Changed lines of the file:
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@@
 <plain>
 <text x="86.36" y="-76.2" size="2.54" layer="94">cc-by-sa</text>
-<text x="86.36" y="-81.28" size="2.54" layer="94">Olivier Gillet</text>
-<text x="86.36" y="-86.36" size="2.54" layer="94">ol.gillet@gmail.com</text>
+<text x="86.36" y="-80.518" size="2.54" layer="94">Codex-Modulex</text>
+<text x="86.36" y="-84.836" size="2.54" layer="94">info@codex-modulex.com</text>
 <text x="144.78" y="66.04" size="1.778" layer="97">mini JTAG</text>
 <text x="142.24" y="-76.2" size="2.54" layer="94">Digital section</text>
 <text x="-30.48" y="132.08" size="1.27" layer="97">grounded on v4.0 or above</text>
+<text x="86.36" y="-91.44" size="1.778" layer="94">Original design by:
+Olivier Gillet of Mutable Instruments</text>
 </plain>
 <instances>
@@
 <plain>
 <text x="149.86" y="-30.48" size="2.54" layer="94">cc-by-sa</text>
-<text x="149.86" y="-35.56" size="2.54" layer="94">Olivier Gillet</text>
-<text x="149.86" y="-40.64" size="2.54" layer="94">ol.gillet@gmail.com</text>
+<text x="149.86" y="-34.798" size="2.54" layer="94">Codex-Modulex</text>
+<text x="149.86" y="-39.37" size="2.54" layer="94">info@codex-modulex.com</text>
 <text x="205.74" y="-30.48" size="2.54" layer="94">Analog Section</text>
 <text x="-17.78" y="154.94" size="1.778" layer="97">0 .. 2.5V</text>
@@
 <text x="114.3" y="152.4" size="1.778" layer="97">0 .. 2.5V</text>
 <text x="106.68" y="99.06" size="1.778" layer="97">0 .. 2.5V</text>
+<text x="149.86" y="-45.72" size="1.778" layer="94">Original design by:
+Olivier Gillet of Mutable Instruments</text>
 </plain>
 <instances>
@@
 <text x="81.28" y="53.34" size="1.778" layer="97">200µA</text>
 <text x="142.24" y="-55.88" size="2.54" layer="94">cc-by-sa</text>
-<text x="142.24" y="-60.96" size="2.54" layer="94">Olivier Gillet</text>
-<text x="142.24" y="-66.04" size="2.54" layer="94">ol.gillet@gmail.com</text>
+<text x="142.24" y="-59.944" size="2.54" layer="94">Codex-Modulex</text>
+<text x="142.24" y="-64.516" size="2.54" layer="94">info@codex-modulex.com</text>
 <text x="198.12" y="-55.88" size="2.54" layer="94">Analog Section</text>
+<text x="142.24" y="-71.12" size="1.778" layer="94">Original design by:
+Olivier Gillet of Mutable Instruments</text>
 </plain>
 <instances>
@@
 </drawing>
 <compatibility>
+<note version="6.3" minversion="6.2.2" severity="warning">
+Since Version 6.2.2 text objects can contain more than one line,
+which will not be processed correctly with this version.
+</note>
 <note version="8.2" severity="warning">
 Since Version 8.2, EAGLE supports online libraries. The ids
